File: PAB_V1.kicad_sch (KiCad schematic)
At the start: 67 parts, among them J1 Screw_Terminal_01x02, J10 Conn_01x01, J11 Conn_01x01, J12 Conn_01x01, J13 Conn_01x01, J14 Conn_01x01, J15 Conn_01x01, J16 Conn_01x01, J17 Conn_01x01, J18 Conn_01x01, J19 Conn_01x01, J2 Screw_Terminal_01x06, J20 Conn_01x01, J21 Conn_01x01, J22 Conn_01x01, J23 Conn_01x01, J24 Conn_01x01, J25 Conn_01x01, J3 Conn_01x01, J4 Conn_01x01, J5 Conn_01x01, J6 Conn_01x01, J7 Conn_01x01, J8 Conn_01x01, J9 Conn_01x01, Q1 AO3400A, Q2 AO3400A, Q3 AO3400A, Q4 AO3400A, Q5 AO3400A, SW1 RESET, SW2 BOOT, U1 AP63205WU-7, U2 TPS2116DRL, U3 AP63203WU-7, U4 ESP32-S3-MINI-1-N4R2, U5 CP2102-GMR

Commit message: Added Bulk capacitor, corrected stuff, checked things
Parts:
- removed C2: 10μF, symbol Device:C
- removed R5: 10 KΩ, symbol Device:R_Small_US
- removed R6: 0Ω, symbol Device:R_Small_US
- removed SW1: RESET, symbol Switch:SW_Push
- removed SW2: BOOT, symbol Switch:SW_Push
- added C2: MA25V220M6X8, easyeda2kicad:CAP-SMD_BD6.3-L6.6-W6.6-LS7.3-FD, symbol Button:MA25V220M6X8
- added C3: 10μF, symbol Device:C_Small
- added C4: 100nF, symbol Device:C_Small
- added J26, J27, J28, J29, J30, J31: Conn_01x01, symbol Connector_Generic:Conn_01x01
- added R11, R13, R15, R17, R19: 100KΩ, symbol Device:R_Small
- added R12, R14, R16, R18, R20: 22Ω, symbol Device:R_Small
- added R5: 10KΩ, symbol Device:R_Small
- added R6, R7, R8: 0Ω, symbol Device:R_Small
- added SW1: RESET, Footprint:SW-SMD_4P-L5.2-W5.2-P3.70-LS6.5, symbol Button:4*4*1.7
- added SW2: BOOT, easyeda2kicad:SW-SMD_4P-L5.2-W5.2-P3.70-LS6.5, symbol Button:4*4*1.7
- C12: renamed from C10; footprint (none) -> Capacitor_SMD:C_0201_0603Metric
- C14: renamed from C12; footprint Capacitor_SMD:C_0201_0603Metric -> (none)
- R2: value 5k2 -> 5k1
- renumbered C8 to C10, C9 to C11, C11 to C13, C13 to C15, C14 to C16, C15 to C17, C16 to C18, C17 to C19, C3 to C5, C4 to C6, C5 to C7, C6 to C8, C7 to C9, R8 to R10, R7 to R9
Connections:
- net +12V: now also C2.1, C3.2, C4.2
- net +3.3V: now also R5.2
- net EN: now also R5.1, R6.2
- net GND: now also C2.2, C3.1, C4.1, R11.1, R13.1, R15.1, R17.1, R19.1, SW1.1, SW1.2, SW2.1, SW2.2
- net GPIO1: now also R12.2; no longer Q1.1 (G)
- net GPIO2: now also R14.2; no longer Q2.1 (G)
- net GPIO3: now also R16.2; no longer Q3.1 (G)
- net GPIO4: now also R18.2; no longer Q4.1 (G)
- net GPIO5: now also R20.2; no longer Q5.1 (G)
- net at C14.1: now also R6.1, SW1.3, SW1.4
- net at U4.23 (IO19): now also R7.1
- net at U4.24 (IO20): now also R8.2
- net GPIO39: now reaches U4.35 (IO39)
- net GPIO39: now also J29.1 (Pin_1)
- net GPIO40: now reaches U4.36 (IO40)
- net GPIO40: now also J28.1 (Pin_1)
- net GPIO41: now reaches U4.37 (IO41)
- net GPIO41: now also J27.1 (Pin_1)
- net GPIO42: now reaches U4.38 (IO42)
- net GPIO42: now also J26.1 (Pin_1)
- net at U4.4 (IO0): now also SW2.3, SW2.4
- new net: Q1.1 (G), R11.2, R12.1
- new net: Q2.1 (G), R13.2, R14.1
- new net: Q3.1 (G), R15.2, R16.1
- new net: Q4.1 (G), R17.2, R18.1
- new net: Q5.1 (G), R19.2, R20.1
- new net GPIO19: J31.1 (Pin_1), R7.2
- new net GPIO20: J30.1 (Pin_1), R8.1
- no-connect marks 37 -> 31
Other:
- note added: "Debugging connector"
- note added: "JTAG pins"
- note added: "USB OTG pins"
- moved on the sheet: C5, C6, C7, D1, J10, J11, J12, J13, J14, J15, J16, J17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

Commit message: Correction to basic component value
Parts:
- added C14: 100nF, symbol Device:C_Small
- C10: value 100nf -> 100nF
- C12: footprint Capacitor_SMD:C_0201_0603Metric -> (none)
- C13: value 1uF -> 1μF
- C15: renamed from C14; value 0.1uF -> 100nF
- C17: renamed from C16; value 0.1uF -> 100nF
- C18: renamed from C17; value 1uF -> 1μF
- C19: renamed from C18; value 0.1uF -> 100nF
- C20: renamed from C19; value 0.1uF -> 100nF
- C9: value 10uF -> 10μF
- L1: value 4.7μH1 -> 4.7μH
- L2: value 4.7uH -> 4.7μH
- R1, R2: value 5k1 -> 5.1KΩ
- R10, R9: value 22 -> 22Ω
- R3: renamed from R4; value 24K -> 24KΩ
- R4: renamed from R3; value 24K -> 24KΩ
- renumbered C15 to C16
Connections:
- net EN: now also C14.2
- net GND: now also C14.1
Other:
- moved on the sheet: C13, R5

Commit message: added decoupling capacitors, added capacitor footprint
Parts:
- added C10: 100nF, Capacitor_SMD:C_1206_3216Metric, symbol Device:C_Small
- added C9: 10μF, Capacitor_SMD:C_1206_3216Metric, symbol Device:C_Small
- C1, C3: footprint (none) -> Capacitor_SMD:C_0805_2012Metric; LCSC Part (none) -> C440198
- C11, C12, C6, C7: footprint (none) -> Capacitor_SMD:C_0805_2012Metric; LCSC Part (none) -> C45783
- C13: renamed from C10; footprint (none) -> Capacitor_SMD:C_0603_1608Metric; LCSC Part (none) -> C14663
- C14: renamed from C9; footprint (none) -> Capacitor_SMD:C_0805_2012Metric; LCSC Part (none) -> C440198
- C15: renamed from C18; footprint (none) -> Capacitor_SMD:C_0805_2012Metric; LCSC Part (none) -> C28323
- C16: renamed from C19; footprint (none) -> Capacitor_SMD:C_0603_1608Metric; LCSC Part (none) -> C14663
- C17: renamed from C20; footprint (none) -> Capacitor_SMD:C_0603_1608Metric; LCSC Part (none) -> C14663
- C18: renamed from C13; footprint (none) -> Capacitor_SMD:C_0805_2012Metric; LCSC Part (none) -> C28323
- C19: renamed from C14; footprint (none) -> Capacitor_SMD:C_0603_1608Metric; LCSC Part (none) -> C14663
- C20: renamed from C15; footprint (none) -> Capacitor_SMD:C_0603_1608Metric; LCSC Part (none) -> C14663
- C21: renamed from C16; footprint (none) -> Capacitor_SMD:C_0805_2012Metric; LCSC Part (none) -> C45783
- C22: renamed from C17; footprint (none) -> Capacitor_SMD:C_0603_1608Metric; LCSC Part (none) -> C14663
- C4, C5: footprint (none) -> Capacitor_SMD:C_0603_1608Metric; LCSC Part (none) -> C14663
- C8: value 100μF -> 47μF; footprint (none) -> Capacitor_SMD:C_1206_3216Metric; LCSC Part (none) -> C96123
- J1: LCSC Part (none) -> C8404
- J2: LCSC Part (none) -> C8379
- Q1, Q2, Q3, Q4, Q5: LCSC Part (none) -> C20917
- U2: LCSC Part (none) -> C3235557
Connections:
- net +5V: now also C10.2, C9.2
- net GND: now also C10.1, C9.1

Commit message: filled part/footprint file (proto bom file)
Parts:
- C10: footprint Capacitor_SMD:C_1206_3216Metric -> Capacitor_SMD:C_0603_1608Metric; LCSC Part C96123 -> C14663
- C2: footprint easyeda2kicad:CAP-SMD_BD6.3-L6.6-W6.6-LS7.3-FD -> Footprint:CAP-SMD_BD6.3-L6.6-W6.6-LS7.3-FD
- C9: footprint Capacitor_SMD:C_1206_3216Metric -> Capacitor_SMD:C_0805_2012Metric; LCSC Part C96123 -> C440198
- J10, J11, J12, J13, J14, J15, J16, J17, J18, J19, J20, J21, J22, J23, J24, J25, J26, J27, J28, J29, J3, J30, J31, J4, J5, J6, J7, J8, J9: footprint (none) -> TestPoint:TestPoint_THTPad_D2.0mm_Drill1.0mm
- L1, L2: footprint (none) -> Inductor_SMD:L_TechFuse_SL0420; LCSC Part (none) -> C22463808
- R1, R2: footprint (none) -> Capacitor_SMD:C_0603_1608Metric; LCSC Part (none) -> C23186
- R10, R12, R14, R16, R18, R20, R9: footprint (none) -> Capacitor_SMD:C_0603_1608Metric; LCSC Part (none) -> C23345
- R11, R13, R15, R17, R19: footprint (none) -> Capacitor_SMD:C_0603_1608Metric; LCSC Part (none) -> C25803
- R3, R4: footprint (none) -> Capacitor_SMD:C_0603_1608Metric; LCSC Part (none) -> C23352
- R5: footprint (none) -> Capacitor_SMD:C_0603_1608Metric; LCSC Part (none) -> C25804
- R6, R7, R8: footprint (none) -> Capacitor_SMD:C_0603_1608Metric; LCSC Part (none) -> C21189
- SW2: footprint easyeda2kicad:SW-SMD_4P-L5.2-W5.2-P3.70-LS6.5 -> Footprint:SW-SMD_4P-L5.2-W5.2-P3.70-LS6.5

Commit message: resolving error, added bom file
Parts:
- D1: value SMBJ15CA_C78809 -> SMBJ15CA
- D2: value TPD4E05U06DQAR_C138714 -> TPD4E05U06DQAR
- R1, R10, R11, R12, R13, R14, R15, R16, R17, R18, R19, R2, R20, R3, R4, R5, R6, R7, R8, R9: footprint Capacitor_SMD:C_0603_1608Metric -> Resistor_SMD:R_0603_1608Metric
Changed lines of the file:
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@@
 			)
 		)
-		(property "Footprint" "Capacitor_SMD:C_0603_1608Metric"
+		(property "Footprint" "Resistor_SMD:R_0603_1608Metric"
 			(at 309.88 55.88 0)
 			(effects
@@
 			)
 		)
-		(property "Footprint" "Capacitor_SMD:C_0603_1608Metric"
+		(property "Footprint" "Resistor_SMD:R_0603_1608Metric"
 			(at 184.15 74.93 0)
 			(effects
@@
 			)
 		)
-		(property "Footprint" "Capacitor_SMD:C_0603_1608Metric"
+		(property "Footprint" "Resistor_SMD:R_0603_1608Metric"
 			(at 252.73 101.6 0)
 			(effects
@@
 			)
 		)
-		(property "Footprint" "Capacitor_SMD:C_0603_1608Metric"
+		(property "Footprint" "Resistor_SMD:R_0603_1608Metric"
 			(at 351.79 41.91 0)
 			(effects
@@
 			)
 		)
-		(property "Footprint" "Capacitor_SMD:C_0603_1608Metric"
+		(property "Footprint" "Resistor_SMD:R_0603_1608Metric"
 			(at 370.84 55.88 0)
 			(effects
@@
 			)
 		)
-		(property "Footprint" "Capacitor_SMD:C_0603_1608Metric"
+		(property "Footprint" "Resistor_SMD:R_0603_1608Metric"
 			(at 74.93 34.29 0)
 			(effects
@@
 			)
 		)
-		(property "Footprint" "Capacitor_SMD:C_0603_1608Metric"
+		(property "Footprint" "Resistor_SMD:R_0603_1608Metric"
 			(at 370.84 41.91 0)
 			(effects
@@
 			)
 		)
-		(property "Footprint" "Capacitor_SMD:C_0603_1608Metric"
+		(property "Footprint" "Resistor_SMD:R_0603_1608Metric"
 			(at 331.47 41.91 0)
 			(effects
@@
 			)
 		)
-		(property "Footprint" "Capacitor_SMD:C_0603_1608Metric"
+		(property "Footprint" "Resistor_SMD:R_0603_1608Metric"
 			(at 204.47 73.66 0)
 			(effects
@@
 			)
 		)
-		(property "Footprint" "Capacitor_SMD:C_0603_1608Metric"
+		(property "Footprint" "Resistor_SMD:R_0603_1608Metric"
 			(at 64.77 242.57 0)
 			(effects
@@
 			)
 		)
-		(property "Footprint" "Capacitor_SMD:C_0603_1608Metric"
+		(property "Footprint" "Resistor_SMD:R_0603_1608Metric"
 			(at 82.55 34.29 0)
 			(effects
@@
 			)
 		)
-		(property "Value" "TPD4E05U06DQAR_C138714"
+		(property "Value" "TPD4E05U06DQAR"
 			(at 106.68 36.83 0)
 			(effects
@@
 			)
 		)
-		(property "Value" "SMBJ15CA_C78809"
+		(property "Value" "SMBJ15CA"
 			(at 55.88 123.698 90)
 			(effects
@@
 			)
 		)
-		(property "Footprint" "Capacitor_SMD:C_0603_1608Metric"
+		(property "Footprint" "Resistor_SMD:R_0603_1608Metric"
 			(at 58.42 252.73 0)
 			(effects
@@
 			)
 		)
-		(property "Footprint" "Capacitor_SMD:C_0603_1608Metric"
+		(property "Footprint" "Resistor_SMD:R_0603_1608Metric"
 			(at 391.16 55.88 0)
 			(effects
@@
 			)
 		)
-		(property "Footprint" "Capacitor_SMD:C_0603_1608Metric"
+		(property "Footprint" "Resistor_SMD:R_0603_1608Metric"
 			(at 252.73 99.06 0)
 			(effects
@@
 			)
 		)
-		(property "Footprint" "Capacitor_SMD:C_0603_1608Metric"
+		(property "Footprint" "Resistor_SMD:R_0603_1608Metric"
 			(at 274.32 231.14 0)
 			(effects
@@
 			)
 		)
-		(property "Footprint" "Capacitor_SMD:C_0603_1608Metric"
+		(property "Footprint" "Resistor_SMD:R_0603_1608Metric"
 			(at 351.79 55.88 0)
 			(effects
@@
 			)
 		)
-		(property "Footprint" "Capacitor_SMD:C_0603_1608Metric"
+		(property "Footprint" "Resistor_SMD:R_0603_1608Metric"
 			(at 331.47 55.88 0)
 			(effects
@@
 			)
 		)
-		(property "Footprint" "Capacitor_SMD:C_0603_1608Metric"
+		(property "Footprint" "Resistor_SMD:R_0603_1608Metric"
 			(at 309.88 41.91 0)
 			(effects
@@
 			)
 		)
-		(property "Footprint" "Capacitor_SMD:C_0603_1608Metric"
+		(property "Footprint" "Resistor_SMD:R_0603_1608Metric"
 			(at 276.86 231.14 0)
 			(effects
@@
 			)
 		)
-		(property "Footprint" "Capacitor_SMD:C_0603_1608Metric"
+		(property "Footprint" "Resistor_SMD:R_0603_1608Metric"
 			(at 391.16 41.91 0)
 			(effects

Commit message: organized netclasses
Connections:
- net USB_DN: now also R10.2, U5.5 (D-)
- net USB_DP: now also R9.1, U5.4 (D+)
- net BOOT: now reaches SW2.3, SW2.4, U4.4 (IO0)
- net Blue_N renamed Blue
- net C_White_N renamed C_White
- net Green_N renamed Green
- net Red_N renamed Red
- net W_White_N renamed W_White
Changed lines of the file:
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@@
+		)
+	)
+	(label "BOOT"
+		(at 241.3 50.8 0)
+		(effects
+			(font
+				(size 1.27 1.27)
+			)
+			(justify left bottom)
 		)
 	)
@@
 		)
 	)
+	(label "USB_DP"
+		(at 267.97 219.71 0)
+		(effects
+			(font
+				(size 1.27 1.27)
+			)
+			(justify left bottom)
+		)
+	)
 	(label "USB_D+"
 		(at 336.55 222.25 180)
@@
 		)
 	)
+	(label "USB_DN"
+		(at 267.97 217.17 0)
+		(effects
+			(font
+				(size 1.27 1.27)
+			)
+			(justify left bottom)
+		)
+	)
 	(label "TCK"
 		(at 330.2 213.36 0)
@@
 		)
 	)
-	(global_label "Blue_N"
+	(global_label "Blue"
 		(shape bidirectional)
 		(at 342.9 107.95 180)
@@
 		)
 		(property "Intersheetrefs" "${INTERSHEET_REFS}"
-			(at 332.3326 107.95 0)
+			(at 334.6307 107.95 0)
 			(effects
 				(font
@@
 		)
 	)
-	(global_label "Green_N"
+	(global_label "Green"
 		(shape bidirectional)
 		(at 339.09 40.64 90)
@@
 		)
 		(property "Intersheetrefs" "${INTERSHEET_REFS}"
-			(at 339.09 28.863 90)
+			(at 339.09 31.1611 90)
 			(effects
 				(font
@@
 		)
 	)
-	(global_label "C_White_N"
+	(global_label "C_White"
 		(shape bidirectional)
 		(at 398.78 40.64 90)
@@
 		)
 		(property "Intersheetrefs" "${INTERSHEET_REFS}"
-			(at 398.78 26.9883 90)
+			(at 398.78 29.2864 90)
 			(effects
 				(font
@@
 		)
 	)
-	(global_label "C_White_N"
+	(global_label "C_White"
 		(shape bidirectional)
 		(at 342.9 113.03 180)
@@
 		)
 		(property "Intersheetrefs" "${INTERSHEET_REFS}"
-			(at 329.2483 113.03 0)
+			(at 331.5464 113.03 0)
 			(effects
 				(font
@@
 		)
 	)
-	(global_label "W_White_N"
+	(global_label "W_White"
 		(shape bidirectional)
 		(at 378.46 40.64 90)
@@
 		)
 		(property "Intersheetrefs" "${INTERSHEET_REFS}"
-			(at 378.46 26.8069 90)
+			(at 378.46 29.105 90)
 			(effects
 				(font
@@
 		)
 	)
-	(global_label "Green_N"
+	(global_label "Green"
 		(shape bidirectional)
 		(at 342.9 102.87 180)
@@
 		)
 		(property "Intersheetrefs" "${INTERSHEET_REFS}"
-			(at 331.123 102.87 0)
+			(at 333.4211 102.87 0)
 			(effects
 				(font
@@
 		)
 	)
-	(global_label "Red_N"
+	(global_label "Red"
 		(shape bidirectional)
 		(at 317.5 40.64 90)
@@
 		)
 		(property "Intersheetrefs" "${INTERSHEET_REFS}"
-			(at 317.5 30.7378 90)
+			(at 317.5 33.0359 90)
 			(effects
 				(font
@@
 		)
 	)
-	(global_label "W_White_N"
+	(global_label "W_White"
 		(shape bidirectional)
 		(at 342.9 110.49 180)
@@
 		)
 		(property "Intersheetrefs" "${INTERSHEET_REFS}"
-			(at 329.0669 110.49 0)
+			(at 331.365 110.49 0)
 			(effects
 				(font
@@
 		)
 	)
-	(global_label "Red_N"
+	(global_label "Red"
 		(shape bidirectional)
 		(at 342.9 105.41 180)
@@
 		)
 		(property "Intersheetrefs" "${INTERSHEET_REFS}"
-			(at 332.9978 105.41 0)
+			(at 335.2959 105.41 0)
 			(effects
 				(font
@@
 		)
 	)
-	(global_label "Blue_N"
+	(global_label "Blue"
 		(shape bidirectional)
 		(at 359.41 40.64 90)
@@
 		)
 		(property "Intersheetrefs" "${INTERSHEET_REFS}"
-			(at 359.41 30.0726 90)
-			(effects
-				(font
+			(at 359.41 32.3707 90)
+			(effects
+				(font

Commit message: starting placing component
Connections:
- net +12V: now also J1.1 (Pin_1), J2.6 (Pin_6); no longer J1.2 (Pin_2), J2.1 (Pin_1)
- net Blue: now also J2.3 (Pin_3); no longer J2.4 (Pin_4)
- net C_White: now also J2.1 (Pin_1); no longer J2.6 (Pin_6)
- net GND: now also J1.2 (Pin_2); no longer J1.1 (Pin_1)
- net GPIO1: now also R20.2; no longer R12.2
- net GPIO2: now also R18.2; no longer R14.2
- net GPIO4: now also R12.2; no longer R18.2
- net GPIO5: now also R14.2; no longer R20.2
- net Green: now also J2.5 (Pin_5); no longer J2.2 (Pin_2)
- net Red: now also J2.4 (Pin_4); no longer J2.3 (Pin_3)
- net W_White: now also J2.2 (Pin_2); no longer J2.5 (Pin_5)
Other:
- moved on the sheet: C2, D1, J1

Commit message: going on with PCB design
Connections:
- net EN: no longer C19.2
- net GND: no longer C19.1
- net USB_DN: now also D2.1 (D1+), D2.10 (NC); no longer D2.2 (D1-)
- net USB_DP: now also D2.2 (D1-), D2.9 (NC); no longer D2.1 (D1+)
Other:
- moved on the sheet: C19, D2
