File: PAB_V1.kicad_sch (KiCad schematic)
At the start: 90 parts, among them J1 Screw_Terminal_01x02, J10 Conn_01x01, J11 Conn_01x01, J12 Conn_01x01, J13 Conn_01x01, J14 Conn_01x01, J15 Conn_01x01, J16 Conn_01x01, J17 Conn_01x01, J18 Conn_01x01, J19 Conn_01x01, J2 Screw_Terminal_01x06, J20 Conn_01x01, J21 Conn_01x01, J22 Conn_01x01, J23 Conn_01x01, J24 Conn_01x01, J25 Conn_01x01, J26 Conn_01x01, J27 Conn_01x01, J28 Conn_01x01, J29 Conn_01x01, J3 Conn_01x01, J30 Conn_01x01, J31 Conn_01x01, J4 Conn_01x01, J5 Conn_01x01, J6 Conn_01x01, J7 Conn_01x01, J8 Conn_01x01, J9 Conn_01x01, Q1 AO3400A, Q2 AO3400A, Q3 AO3400A, Q4 AO3400A, Q5 AO3400A, SW1 RESET, SW2 BOOT, U1 AP63205WU-7, U2 TPS2116DRL, U3 AP63203WU-7, U4 ESP32-S3-MINI-1-N4R2, U5 CP2102-GMR

Commit message: going on with pcb layout
Parts:
- added J32: Conn_01x01, TestPoint:TestPoint_THTPad_D2.0mm_Drill1.0mm, symbol Connector_Generic:Conn_01x01
Connections:
- net +5V_USB: no longer C1.1, D2.4 (D2+), USB1.A4B9 (VBUS), USB1.B4A9 (VBUS)
- net USB_DN: now also D2.2 (D1-), D2.9 (NC); no longer D2.1 (D1+), D2.10 (NC)
- net USB_DP: now also D2.1 (D1+), D2.10 (NC); no longer D2.2 (D1-), D2.9 (NC)
- net at D2.7 (NC): now also C1.1, D2.4 (D2+), USB1.A4B9 (VBUS), USB1.B4A9 (VBUS)
- no-connect marks 31 -> 28

Commit message: going on with connections
Parts:
- added J33, J34, J35: Conn_01x01, TestPoint:TestPoint_THTPad_D2.0mm_Drill1.0mm, symbol Connector_Generic:Conn_01x01
Connections:
- net +3.3V: now also J32.1 (Pin_1)
- net +5V: now also J33.1 (Pin_1)
- net +5V_USB: now also C1.1, D2.4 (D2+), D2.7 (NC), USB1.A4B9 (VBUS), USB1.B4A9 (VBUS)
- net EN: now also C19.1
- net GND: now also C19.2, J34.1 (Pin_1), J35.1 (Pin_1); no longer SW2.1
- no-connect marks 28 -> 29
Other:
- moved on the sheet: C19, J26, J27, J28, J29, J30, J31, J32
