File: PAB_V1.kicad_pcb (KiCad board)
At the start: 4 copper layers, 90 parts, among them J1 Screw_Terminal_01x02, J10 Conn_01x01, J11 Conn_01x01, J12 Conn_01x01, J13 Conn_01x01, J14 Conn_01x01, J15 Conn_01x01, J16 Conn_01x01, J17 Conn_01x01, J18 Conn_01x01, J19 Conn_01x01, J2 Screw_Terminal_01x06, J20 Conn_01x01, J21 Conn_01x01, J22 Conn_01x01, J23 Conn_01x01, J24 Conn_01x01, J25 Conn_01x01, J26 Conn_01x01, J27 Conn_01x01, J28 Conn_01x01, J29 Conn_01x01, J3 Conn_01x01, J30 Conn_01x01, J31 Conn_01x01, J4 Conn_01x01, J5 Conn_01x01, J6 Conn_01x01, J7 Conn_01x01, J8 Conn_01x01, J9 Conn_01x01, Q1 AO3400A, Q2 AO3400A, Q3 AO3400A, Q4 AO3400A, Q5 AO3400A, SW1 RESET, SW2 BOOT, U1 AP63205WU-7, U2 TPS2116DRL, U3 AP63203WU-7, U4 ESP32-S3-MINI-1-N4R2, U5 CP2102-GMR

Commit message: starting placing component
Parts:
- moved USB1 151.6 mm to (113.8, 97.2), turned to -90 degrees
- moved U5 142.1 mm to (123.2, 109.5), turned to 180 degrees
- moved J1 140.4 mm to (133.2, 66.2), turned to -90 degrees
- moved D2 140.4 mm to (122.2, 102.7), turned to 180 degrees
- moved R1 134.9 mm to (119.2, 89.8), turned to 90 degrees
- moved R2 132.7 mm to (122.2, 89.8), turned to 90 degrees
- moved C16 130.0 mm to (118.0, 106.8), turned to 90 degrees
- moved L1 129.3 mm to (137.1, 93.5), turned to 90 degrees
- moved D1 128.4 mm to (133.2, 72.8)
- moved C19 123.9 mm to (122.5, 121.5), turned to 90 degrees
- moved R14 117.3 mm to (149.8, 82.8), turned to -90 degrees
- moved R13 117.3 mm to (150.4, 79.1), turned to 180 degrees
- moved C4 116.6 mm to (134.6, 86.5), turned to 90 degrees
- moved L2 115.6 mm to (152.5, 95.0)
- moved SW1 113.2 mm to (125.5, 131.2)
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Connections:
- J1 pad 1: GND -> +12V
- J1 pad 2: +12V -> GND
- J2 pad 1: +12V -> C_White
- J2 pad 2: Green -> W_White
- J2 pad 3: Red -> Blue
- J2 pad 4: Blue -> Red
- J2 pad 5: W_White -> Green
- J2 pad 6: C_White -> +12V
- R12 pad 2: GPIO1 -> GPIO4
- R14 pad 2: GPIO2 -> GPIO5
- R18 pad 2: GPIO4 -> GPIO2
- R20 pad 2: GPIO5 -> GPIO1

Commit message: going on with PCB design
Parts:
- added .: MountingHole_2.5mm, MountingHole:MountingHole_2.5mm, F.Cu at (149.4, 98.0)
- moved C17 128.1 mm to (122.7, 111.0)
- moved R10 126.0 mm to (127.8, 110.7), turned to 90 degrees
- moved R9 123.7 mm to (129.8, 110.7), turned to 90 degrees
- moved R4 120.3 mm to (133.9, 98.8), turned to 90 degrees
- moved R3 120.0 mm to (133.9, 102.4), turned to 90 degrees
- moved R5 117.2 mm to (135.4, 125.4), turned to 90 degrees
- moved C20 109.8 mm to (131.8, 127.5), turned to 90 degrees
- moved R8 98.3 mm to (156.2, 112.5), turned to 180 degrees
- moved R7 98.0 mm to (156.5, 110.2), turned to 180 degrees
- moved J27 93.8 mm to (174.0, 101.6), turned to 180 degrees
- moved J22 92.9 mm to (174.0, 112.0)
- moved J23 92.2 mm to (174.0, 114.6)
- moved J28 91.4 mm to (174.0, 99.1), turned to 180 degrees
- moved J29 89.4 mm to (174.0, 96.5), turned to 180 degrees
- moved J24 88.3 mm to (174.0, 109.2), turned to 180 degrees
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Connections:
- C19 pad 1: GND -> unconnected-(C19-Pad1)
- C19 pad 2: /EN -> unconnected-(C19-Pad2)
- D2 pad 1: USB_DP -> USB_DN
- D2 pad 10: unconnected-(D2-NC-Pad10) -> USB_DN
- D2 pad 2: USB_DN -> USB_DP
- D2 pad 9: unconnected-(D2-NC-Pad9) -> USB_DP
Routing:
- net +5V_USB: track 0.00 -> 18.7 mm, vias 0 -> 5
- net USB_DP: track 0.00 -> 16.4 mm, vias 0 -> 1
- net USB_DN: track 0.00 -> 15.1 mm, vias 0 -> 1
- net /EN: track 0.00 -> 12.3 mm
- net +5V_PS: track 0.00 -> 11.9 mm
- net W_White: track 0.00 -> 8.67 mm
- net Red: track 0.00 -> 8.67 mm
- net Green: track 0.00 -> 8.67 mm
- net C_White: track 0.00 -> 8.67 mm
- net Blue: track 0.00 -> 8.67 mm
- net Net-(U3-SW): track 0.00 -> 5.30 mm
- net Net-(C20-Pad1): track 0.00 -> 4.49 mm
- net Net-(U2-PR1): track 0.00 -> 3.84 mm
- net Net-(Q2-G): track 0.00 -> 3.45 mm
- net Net-(Q1-G): track 0.00 -> 3.44 mm
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- added copper zone on F.Cu, net +12V
- added copper zone on In2.Cu, net +3.3V
- added copper zone on F.Cu, net +5V
- added copper zone on In2.Cu, net +5V
- added copper zone on In2.Cu, net +5V_USB
- added copper zone on F.Cu, net GND
- added copper zone on In1.Cu, net GND
Other:
- board outline added: 77.1 x 71 mm

Commit message: going on with pcb layout
Parts:
- moved J31 55.1 mm to (137.7, 115.1)
- moved J30 51.5 mm to (140.2, 115.1)
- moved J24 29.8 mm to (181.1, 80.3)
- moved J25 17.5 mm to (174.0, 89.2)
- moved C12 11.4 mm to (144.3, 101.1)
- moved J15 8.89 mm to (181.1, 83.6)
- moved R8 7.89 mm to (148.3, 113.0), turned to -90 degrees
- moved C11 7.00 mm to (144.3, 103.4)
- moved R7 6.71 mm to (150.4, 113.0), turned to 90 degrees
- moved R9 6.01 mm to (124.2, 108.5), turned to 180 degrees
- moved J18 5.33 mm to (174.0, 91.7)
- moved J20 5.33 mm to (174.0, 96.8)
- moved J21 5.33 mm to (174.0, 99.4)
- moved J26 5.33 mm to (174.0, 109.5)
- moved J27 5.33 mm to (174.0, 106.9)
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Connections:
- C1 pad 1: +5V_USB -> Net-(D2-D2+)
- D2 pad 1: USB_DN -> USB_DP
- D2 pad 10: USB_DN -> USB_DP
- D2 pad 2: USB_DP -> USB_DN
- D2 pad 4: +5V_USB -> Net-(D2-D2+)
- D2 pad 7: unconnected-(D2-NC-Pad7) -> Net-(D2-D2+)
- D2 pad 9: USB_DP -> USB_DN
- USB1 pad A4B9: +5V_USB -> Net-(D2-D2+)
- USB1 pad B4A9: +5V_USB -> Net-(D2-D2+)
Routing:
- net GPIO17: track 0.00 -> 61.4 mm, vias 0 -> 1
- net GPIO18: track 0.00 -> 60.1 mm, vias 0 -> 1
- net GPIO21: track 0.00 -> 59.3 mm, vias 0 -> 1
- net GPIO47: track 0.00 -> 59.1 mm, vias 0 -> 1
- net GPIO26: track 0.00 -> 58.7 mm, vias 0 -> 1
- net GPIO5: track 0.47 -> 51.8 mm
- net GPIO4: track 0.39 -> 51.1 mm
- net GPIO33: track 0.00 -> 50.3 mm, vias 0 -> 1
- net GPIO3: track 0.39 -> 50.3 mm
- net GPIO2: track 0.30 -> 49.2 mm
- net GPIO14: track 0.00 -> 48.7 mm, vias 0 -> 2
- net GPIO1: track 0.32 -> 48.5 mm
- net GPIO34: track 0.00 -> 46.9 mm, vias 0 -> 1
- net GPIO13: track 0.00 -> 46.6 mm, vias 0 -> 1
- net GPIO12: track 0.00 -> 44.1 mm, vias 0 -> 1
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
Commit message: going on with connections
Parts:
- added J32: Conn_01x01, TestPoint:TestPoint_THTPad_D2.0mm_Drill1.0mm, F.Cu at (144.3, 96.5)
- added J33: Conn_01x01, TestPoint:TestPoint_THTPad_D2.0mm_Drill1.0mm, F.Cu at (118.1, 116.8)
- added J34: Conn_01x01, TestPoint:TestPoint_THTPad_D2.0mm_Drill1.0mm, F.Cu at (120.4, 121.9)
- added J35: Conn_01x01, TestPoint:TestPoint_THTPad_D2.0mm_Drill1.0mm, F.Cu at (174.0, 81.3)
- moved R2 9.66 mm to (123.2, 105.5), turned to 0 degrees
- moved D2 8.12 mm to (118.6, 110.8), turned to -90 degrees
- moved R1 7.39 mm to (123.2, 102.6), turned to 0 degrees
- moved R3 1.63 mm to (134.9, 101.1), turned to 180 degrees
- moved SW2 1.14 mm to (168.9, 126.7), turned to 180 degrees
- moved J24 0.80 mm to (181.4, 81.0)
- moved J15 0.36 mm to (181.4, 83.8)
- turned C19 to 90 degrees
Connections:
- C1 pad 1: Net-(D2-D2+) -> +5V_USB
- C19 pad 1: unconnected-(C19-Pad1) -> /EN
- C19 pad 2: unconnected-(C19-Pad2) -> GND
- D2 pad 4: Net-(D2-D2+) -> +5V_USB
- D2 pad 7: Net-(D2-D2+) -> +5V_USB
- SW2 pad 1: GND -> unconnected-(SW2-Pad1)
- USB1 pad A4B9: Net-(D2-D2+) -> +5V_USB
- USB1 pad B4A9: Net-(D2-D2+) -> +5V_USB
Routing:
- net +3.3V: track 0.00 -> 23.0 mm, vias 0 -> 17
- net /BOOT: track 0.00 -> 16.4 mm
- net +5V_PS: track 11.9 -> 25.1 mm, vias 0 -> 2
- net Net-(C20-Pad1): track 4.49 -> 10.7 mm
- net GND: track 8.64 -> 2.47 mm, vias 36 -> 64
- net GPIO21: track 59.3 -> 65.2 mm
- net GPIO18: track 60.1 -> 66.0 mm
- net Net-(U1-SW): track 0.00 -> 5.36 mm
- net GPIO17: track 61.4 -> 66.3 mm
- net GPIO26: track 58.7 -> 63.0 mm
- net Net-(U5-VDD): track 0.00 -> 4.11 mm
- net GPIO47: track 59.1 -> 62.6 mm
- net Net-(USB1-CC2): track 0.00 -> 3.47 mm
- net Net-(USB1-CC1): track 0.00 -> 3.15 mm
- net Net-(D2-D2+): track 2.40 -> 0.00 mm, vias 2 -> 0
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- added copper zone on F.Cu, net +3.3V
