File: PAB_V1.kicad_pcb (KiCad board)
At the start: 4 copper layers, 77.1 x 71 mm, 95 parts, among them J1 Screw_Terminal_01x02, J10 Conn_01x01, J11 Conn_01x01, J12 Conn_01x01, J13 Conn_01x01, J14 Conn_01x01, J15 Conn_01x01, J16 Conn_01x01, J17 Conn_01x01, J18 Conn_01x01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

Commit message: reorganized text layout
Parts:
- moved IO38 0.12 mm to (174.0, 99.5)
- moved IO46 0.05 mm to (174.0, 114.5)
- renumbered J32 to 3.3V, J33 to 5V, SW2 to BOOT, J35 to GND, J34 to GND, J7 to IO10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
